Commit message: modify for lecture

File: open_manipulator_description/urdf/open_manipulator.urdf.xacro (robot description, xacro)
@@ -29,5 +29,5 @@
     <parent link="link1"/>
     <child link="link2"/>
-    <origin xyz="0.012 0.0 0.017" rpy="0 0 0"/>
+    <origin xyz="0.012 0.0 0.0275" rpy="0 0 0"/>
     <axis xyz="0 0 1"/>
     <limit velocity="4.8" effort="1" lower="${-pi*0.9}" upper="${pi*0.9}" />
@@ -60,5 +60,5 @@
     <parent link="link2"/>
     <child link="link3"/>
-    <origin xyz="0.0 0.0 0.0595" rpy="0 0 0"/>
+    <origin xyz="0.0 0.0 0.040" rpy="0 0 0"/>
     <axis xyz="0 1 0"/>
     <limit velocity="4.8" effort="1" lower="${-pi*0.57}" upper="${pi*0.5}" />
@@ -91,5 +91,5 @@
     <parent link="link3"/>
     <child link="link4"/>
-    <origin xyz="0.024 0 0.128" rpy="0 0 0"/>
+    <origin xyz="0.025 0 0.084" rpy="0 0 0"/>
     <axis xyz="0 1 0"/>
     <limit velocity="4.8" effort="1" lower="${-pi*0.3}" upper="${pi*0.44}" />
@@ -122,5 +122,5 @@
     <parent link="link4"/>
     <child link="link5"/>
-    <origin xyz="0.124 0.0 0.0" rpy="0 0 0"/>
+    <origin xyz="0.082 0.0 0.0" rpy="0 0 0"/>
     <axis xyz="0 1 0"/>
     <limit velocity="4.8" effort="1" lower="${-pi*0.57}" upper="${pi*0.65}" />
@@ -150,4 +150,5 @@
   </link>
   <!--  Gripper joint -->
+  <!-- TODO adjust origin of gripper for mini manipulator-->
   <joint name="gripper" type="prismatic">
     <parent link="link5"/>
